Commit message: edit world

File: raspimouse_gazebo/materials/sample_maze.wall.xacro (robot description, xacro)
@@ -1,8 +1,9 @@
 <?xml version="1.0" ?>
 <sdf version="1.4" xmlns:xacro="http://ros.org/wiki/xacro">
-  <xacro:macro name="wall" params="*pose">
-    <model name='wall'>
+  <xacro:macro name="wall" params="pose name">
+    <model name="${name}">
       <!-- <pose>&#45;0.09 0 0.5 0 0 1.57</pose> -->
-      <xacro:insert_block name="pose" />
+      <!-- <xacro:insert_block name="pose" /> -->
+      <pose>${pose}</pose>
       <link name='link'>
         <inertial>

File: raspimouse_gazebo/materials/sample_maze.world.xacro (robot description, xacro)
@@ -4,7 +4,7 @@
 <xacro:include filename="$(find raspimouse_gazebo)/materials/sample_maze.wall.xacro" />
 <world name="default">
-  <xacro:include>
+  <!-- <xacro:include>
     <uri>model://ground_plane</uri>
-  </xacro:include>
+  </xacro:include> -->
   <light name='sun' type='directional'>
     <cast_shadows>1</cast_shadows>
@@ -33,56 +33,24 @@
   </gui>
   <!-- horizontal -->
-  <xacro:wall>
-    <pose>-0.090 0.006 0.025 0 0 1.57</pose>
-  </xacro:wall>
-  <xacro:wall>
-    <pose>-0.090 -0.174 0.025 0 0 1.57</pose>
-  </xacro:wall>
-  <xacro:wall>
-    <pose>-0.090 -0.354 0.025 0 0 1.57</pose>
-  </xacro:wall>
+  <xacro:wall pose="-0.090 0.006 0.025 0 0 1.57" name="wall1"/>
+  <xacro:wall pose="-0.090 -0.174 0.025 0 0 1.57" name="wall1"/>
+  <xacro:wall pose="-0.090 -0.354 0.025 0 0 1.57" name="wall1"/>
   <!-- vertical -->
-  <xacro:wall>
-    <pose>0.006 0.090 0.025 0 0 0</pose>
-  </xacro:wall>
-  <xacro:wall>
-    <pose>0.186 0.090 0.025 0 0 0</pose>
-  </xacro:wall>
-  <xacro:wall>
-    <pose>0.366 0.090 0.025 0 0 0</pose>
-  </xacro:wall>
+  <xacro:wall pose="0.006 0.090 0.025 0 0 0" name="wall1"/>
+  <xacro:wall pose="0.186 0.090 0.025 0 0 0" name="wall1"/>
+  <xacro:wall pose="0.366 0.090 0.025 0 0 0" name="wall1"/>
   <!-- horizontal -->
-  <xacro:wall>
-    <pose>0.450 0.006 0.025 0 0 1.57</pose>
-  </xacro:wall>
-  <xacro:wall>
-    <pose>0.450 -0.174 0.025 0 0 1.57</pose>
-  </xacro:wall>
-  <xacro:wall>
-    <pose>0.450 -0.354 0.025 0 0 1.57</pose>
-  </xacro:wall>
+  <xacro:wall pose="0.450 0.006 0.025 0 0 1.57" name="wall1"/>
+  <xacro:wall pose="0.450 -0.174 0.025 0 0 1.57" name="wall1"/>
+  <xacro:wall pose="0.450 -0.354 0.025 0 0 1.57" name="wall1"/>
   <!-- vertical -->
-  <xacro:wall>
-    <pose>0.006 -0.450 0.025 0 0 0</pose>
-  </xacro:wall>
-  <xacro:wall>
-    <pose>0.186 -0.450 0.025 0 0 0</pose>
-  </xacro:wall>
-  <xacro:wall>
-    <pose>0.366 -0.450 0.025 0 0 0</pose>
-  </xacro:wall>
+  <xacro:wall pose="0.006 -0.450 0.025 0 0 0" name="wall1"/>
+  <xacro:wall pose="0.186 -0.450 0.025 0 0 0" name="wall1"/>
+  <xacro:wall pose="0.366 -0.450 0.025 0 0 0" name="wall1"/>
   <!-- plus alpha -->
-  <xacro:wall>
-    <pose>0.186 -0.270 0.025 0 0 0</pose>
-  </xacro:wall>
-  <xacro:wall>
-    <pose>0.366 -0.090 0.025 0 0 0</pose>
-  </xacro:wall>
-  <xacro:wall>
-    <pose>0.270 -0.174 0.025 0 0 1.57</pose>
-  </xacro:wall>
-  <xacro:wall>
-    <pose>0.006 -0.090 0.025 0 0 0</pose>
-  </xacro:wall>
+  <xacro:wall pose="0.186 -0.270 0.025 0 0 0" name="wall1"/>
+  <xacro:wall pose="0.366 -0.090 0.025 0 0 0" name="wall1"/>
+  <xacro:wall pose="0.270 -0.174 0.025 0 0 1.57" name="wall1"/>
+  <xacro:wall pose="0.006 -0.090 0.025 0 0 0" name="wall1"/>
 </world>
 </sdf>
