Commit message: 車体と車輪のurdf変更
車輪・車体の重さ、イナーシャの変更、車輪の向きを変更、読み込むCADデータを自分のデータにする

File: raspimouse_description/robots/raspimouse.urdf.xacro (robot description, xacro)
@@ -12,14 +12,14 @@
   <link name="base_footprint" />
   <xacro:base parent="base_footprint">
-    <origin xyz="0 0 0.00185" />
+    <origin xyz="0 0 0.00185"  rpy="0 0 0"/>
   </xacro:base>
   <!-- Wheel -->
   <xacro:wheel prefix="right" parent="base_link">
-    <origin xyz="0 -0.0425 0.02215" rpy="1.57 0 0" />
-    <axis xyz="0 0 -1" />
+    <origin xyz="0 -0.0475 0.02215" rpy="0 0 3.1416" />
+    <axis xyz="0 -1 0" />
   </xacro:wheel>
   <xacro:wheel prefix="left" parent="base_link">
-    <origin xyz="0 0.0425 0.02215" rpy="-1.57 0 0" />
-    <axis xyz="0 0 1" />
+    <origin xyz="0 0.0475 0.02215" rpy="0 0 0" />
+    <axis xyz="0 1 0" />
   </xacro:wheel>
   <!-- Sensors -->

File: raspimouse_description/robots/raspimouse_urg.urdf.xacro (robot description, xacro)
@@ -13,14 +13,18 @@
   <link name="base_footprint" />
   <xacro:base parent="base_footprint">
-    <origin xyz="0 0 0.00185" />
+    <origin xyz="0 0 0.00185"  rpy="0 0 0"/>
   </xacro:base>
   <!-- Wheel -->
   <xacro:wheel prefix="right" parent="base_link">
-    <origin xyz="0 -0.0425 0.02215" rpy="1.57 0 0" />
-    <axis xyz="0 0 -1" />
+   <!--  <origin xyz="0 -0.0425 0.02215" rpy="1.57 0 0" />-->
+   <!--  <axis xyz="0 0 -1" />-->
+    <origin xyz="0 -0.0475 0.02215" rpy="0 0 3.1416" />
+    <axis xyz="0 -1 0" />
   </xacro:wheel>
   <xacro:wheel prefix="left" parent="base_link">
-    <origin xyz="0 0.0425 0.02215" rpy="-1.57 0 0" />
-    <axis xyz="0 0 1" />
+   <!--  <origin xyz="0 0.0425 0.02215" rpy="-1.57 0 0" />-->
+   <!--  <axis xyz="0 0 1" />-->
+    <origin xyz="0 0.0475 0.02215" rpy="0 0 0" />
+    <axis xyz="0 1 0" />
   </xacro:wheel>
   <!-- Sensors -->

File: raspimouse_description/urdf/body/body.urdf.xacro (robot description, xacro)
@@ -13,10 +13,12 @@
       <visual>
         <geometry>
-          <mesh filename="package://raspimouse_description/meshes/dae/body/RasPiMouse_body.dae" />
+          <!-- <mesh filename="package://raspimouse_description/meshes/dae/body/RasPiMouse_body.dae" /> -->
+          <mesh filename="package://raspimouse_description/meshes/obj/body/raspi_body.obj" />
         </geometry>
       </visual>
       <collision>
         <geometry>
-          <mesh filename="package://raspimouse_description/meshes/dae/body/RasPiMouse_body.dae" />
+          <!-- <mesh filename="package://raspimouse_description/meshes/dae/body/RasPiMouse_body.dae" /> -->
+          <mesh filename="package://raspimouse_description/meshes/obj/body/raspi_body.obj" />
         </geometry>
       </collision>
@@ -29,10 +31,16 @@
         <!-- <origin xyz="&#45;0.005075 &#45;0.000427 0.029879" /> -->
         <!-- virtual origin -->
-        <origin xyz="-0.001 0.0 0.029879" />
-        <mass value="31.20594944"/>
+        <origin xyz="-0.01081720 -0.00078063 0.02842790" />
+        <!-- <origin xyz="-0.001 0.0 0.029879" /> -->
+        <!-- <mass value="31.20594944"/>
         <inertia
               ixx="1.79583172"
               ixy="0.03278618" iyy="1.55345103"
-              ixz="0.02535482" iyz="0.01272625" izz="1.22908514"/>
+              ixz="0.02535482" iyz="0.01272625" izz="1.22908514"/> -->
+        <mass value="0.23409945"/>
+        <inertia
+              ixx="0.00020481"
+              ixy="0.00000162" iyy="0.00025632"
+              ixz="0.00000155" iyz="0.00000742" izz="0.00026763"/>
         <!-- <mass value="0.7186" />
         <inertia ixx="0.001238161833" ixy="0.000000904986" iyy="0.001368529369" ixz="0.000100297310" iyz="0.000022118177" izz="0.000784319117" /> -->

File: raspimouse_description/urdf/body/body_urg.urdf.xacro (robot description, xacro)
@@ -29,14 +29,19 @@
         <!-- <origin xyz="&#45;0.003851 &#45;0.000443 0.031714" /> -->
         <!-- virtual origin -->
-        <origin xyz="-0.000851 -0.000003 0.031714" />
-        <mass value="31.20594944"/>
-          <inertia
+        <!--<origin xyz="-0.000851 -0.000003 0.031714" />-->
+        <origin xyz="-0.01081720 -0.00078063 0.02842790" />
+        <!-- <mass value="31.20594944"/>
+        <inertia
               ixx="1.79583172"
               ixy="0.03278618" iyy="1.55345103"
-              ixz="0.02535482" iyz="0.01272625" izz="1.22908514"/>
-        </inertial>
+              ixz="0.02535482" iyz="0.01272625" izz="1.22908514"/> -->
+        <mass value="0.23409945"/>
+        <inertia
+              ixx="0.00020481"
+              ixy="0.00000162" iyy="0.00025632"
+              ixz="0.00000155" iyz="0.00000742" izz="0.00026763"/>
         <!-- <mass value="0.759881" />
-        <inertia ixx="0.001561279589" ixy="0.00000150035" iyy="0.001698462955" ixz="0.000042679786" iyz="0.000023629024" izz="0.000855782529" />
-      </inertial> -->
+        <inertia ixx="0.001561279589" ixy="0.00000150035" iyy="0.001698462955" ixz="0.000042679786" iyz="0.000023629024" izz="0.000855782529" /> -->
+      </inertial>
     </link>
   </xacro:macro>

File: raspimouse_description/urdf/wheel/wheel.urdf.xacro (robot description, xacro)
@@ -4,5 +4,5 @@
   <xacro:include filename="$(find raspimouse_description)/urdf/wheel/wheel.gazebo.xacro" />
   <xacro:property name="wheel_radius" value="0.024" />
-  <xacro:property name="wheel_length" value="0.01" />
+  <xacro:property name="wheel_length" value="0.008" />
   <xacro:property name="wheel_mass" value="0.0113" />
   <xacro:macro name="wheel" params="prefix parent *joint_origin *joint_axis">
@@ -12,15 +12,17 @@
     <parent link="${parent}" />
     <child link="${prefix}_wheel" />
-    <limit effort="70" velocity="15" />
-    <safety_controller  k_velocity="10" />
-    <dynamics damping="1.0" friction="1.0" />
+    <!-- <limit effort="70" velocity="15" /> -->
+    <!-- <safety_controller  k_velocity="10" /> -->
+    <!-- <dynamics damping="1.0" friction="1.0" /> -->
   </joint>
   <link name="${prefix}_wheel">
     <visual>
       <geometry>
-        <mesh filename="package://raspimouse_description/meshes/dae/wheel/RasPiMouse_wheel.dae" />
+        <!-- <mesh filename="package://raspimouse_description/meshes/dae/wheel/RasPiMouse_wheel.dae" /> -->
+        <mesh filename="package://raspimouse_description/meshes/obj/wheel/raspi_wheel2.obj" />
       </geometry>
     </visual>
     <collision>
+        <origin xyz="0 ${-wheel_length/2.0} 0" rpy="${pi / 2} 0 0" />
         <geometry>
           <cylinder radius="${wheel_radius}" length="${wheel_length}" />
@@ -28,14 +30,20 @@
         </geometry>
     </collision>
-      <inertial>
-        <origin xyz="-0.000107 0 0.002875" />
-        <mass value="3.16354494"/>
-        <inertia
-              ixx="0.02296002"
-              ixy="0.00000000" iyy="0.04452360"
-              ixz="0.00000000" iyz="-0.00000001" izz="0.02296002"/>
-        <!-- <mass value="${wheel_mass}" />
-        <inertia ixx="0.000002208187" ixy="0.000000000001" iyy="0.00000218412" ixz="0.000000004787" iyz="0.000000000003" izz="0.000004078299" /> -->
-      </inertial>
+    <inertial>
+      <!-- <origin xyz="-0.000107 0 0.002875" /> -->
+      <origin xyz="-0.00008176 	-0.00478578 0.00000005" />
+      <!-- <mass value="3.16354494"/>
+      <inertia
+            ixx="0.02296002"
+            ixy="0.00000000" iyy="0.04452360"
+            ixz="0.00000000" iyz="-0.00000001" izz="0.02296002"/> -->
+      <mass value="0.0553656"/>
+      <inertia
+            ixx="0.0000115"
+            ixy="0.0000000" iyy="0.0000223"
+            ixz="0.0000000" iyz="-0.0000000" izz="0.0000114"/>
+      <!-- <mass value="${wheel_mass}" />
+      <inertia ixx="0.000002208187" ixy="0.000000000001" iyy="0.00000218412" ixz="0.000000004787" iyz="0.000000000003" izz="0.000004078299" /> -->
+    </inertial>
   </link>
   </xacro:macro>

Commit message: edit world

File: raspimouse_description/robots/raspimouse.urdf.xacro (robot description, xacro)
@@ -45,4 +45,5 @@
     <plugin name="gazebo_ros_control" filename="libgazebo_ros_control.so">
       <robotNamespace>raspimouse_on_gazebo</robotNamespace>
+      <legacyModeNS>true</legacyModeNS>
     </plugin>
   </gazebo>

File: raspimouse_description/robots/raspimouse_urg.urdf.xacro (robot description, xacro)
@@ -49,4 +49,5 @@
     <plugin name="gazebo_ros_control" filename="libgazebo_ros_control.so">
       <robotNamespace>raspimouse_on_gazebo</robotNamespace>
+      <legacyModeNS>true</legacyModeNS>
     </plugin>
   </gazebo>

File: raspimouse_description/urdf/body/body.gazebo.xacro (robot description, xacro)
@@ -7,5 +7,7 @@
       <!-- <mu2 value="0.05" /> -->
       <mu1>0.05</mu1>
-      <mu2>0.05</mu2>
+      <!-- <mu2>0.05</mu2> -->
+      <kp value="2000000" />
+      <kd value="100" />
     </gazebo>
   </xacro:macro>

File: raspimouse_description/urdf/body/body.urdf.xacro (robot description, xacro)
@@ -30,6 +30,11 @@
         <!-- virtual origin -->
         <origin xyz="-0.001 0.0 0.029879" />
-        <mass value="0.7186" />
-        <inertia ixx="0.001238161833" ixy="0.000000904986" iyy="0.001368529369" ixz="0.000100297310" iyz="0.000022118177" izz="0.000784319117" />
+        <mass value="31.20594944"/>
+        <inertia
+              ixx="1.79583172"
+              ixy="0.03278618" iyy="1.55345103"
+              ixz="0.02535482" iyz="0.01272625" izz="1.22908514"/>
+        <!-- <mass value="0.7186" />
+        <inertia ixx="0.001238161833" ixy="0.000000904986" iyy="0.001368529369" ixz="0.000100297310" iyz="0.000022118177" izz="0.000784319117" /> -->
       </inertial>
     </link>

File: raspimouse_description/urdf/body/body_urg.gazebo.xacro (robot description, xacro)
@@ -7,5 +7,7 @@
       <!-- <mu2 value="0.05" /> -->
       <mu1>0.05</mu1>
-      <mu2>0.05</mu2>
+      <!-- <mu2>0.05</mu2> -->
+      <kp value="2000000" />
+      <kd value="100" />
     </gazebo>
   </xacro:macro>

File: raspimouse_description/urdf/body/body_urg.urdf.xacro (robot description, xacro)
@@ -30,7 +30,13 @@
         <!-- virtual origin -->
         <origin xyz="-0.000851 -0.000003 0.031714" />
-        <mass value="0.759881" />
+        <mass value="31.20594944"/>
+          <inertia
+              ixx="1.79583172"
+              ixy="0.03278618" iyy="1.55345103"
+              ixz="0.02535482" iyz="0.01272625" izz="1.22908514"/>
+        </inertial>
+        <!-- <mass value="0.759881" />
         <inertia ixx="0.001561279589" ixy="0.00000150035" iyy="0.001698462955" ixz="0.000042679786" iyz="0.000023629024" izz="0.000855782529" />
-      </inertial>
+      </inertial> -->
     </link>
   </xacro:macro>

File: raspimouse_description/urdf/wheel/wheel.gazebo.xacro (robot description, xacro)
@@ -5,5 +5,5 @@
       <selfCollide>true</selfCollide>
       <mu1>1.0</mu1>
-      <mu2>1.0</mu2>
+      <!--<mu2>1.0</mu2>-->
       <kp>200000.0</kp>
       <kd>100.0</kd>

File: raspimouse_description/urdf/wheel/wheel.urdf.xacro (robot description, xacro)
@@ -24,12 +24,17 @@
     <collision>
         <geometry>
-          <!-- <cylinder radius="${wheel_radius}" length="${wheel_length}" /> -->
-          <mesh filename="package://raspimouse_description/meshes/dae/wheel/RasPiMouse_wheel.dae" />
+          <cylinder radius="${wheel_radius}" length="${wheel_length}" />
+          <!-- <mesh filename="package://raspimouse_description/meshes/dae/wheel/RasPiMouse_wheel.dae" /> -->
         </geometry>
     </collision>
       <inertial>
         <origin xyz="-0.000107 0 0.002875" />
-        <mass value="${wheel_mass}" />
-        <inertia ixx="0.000002208187" ixy="0.000000000001" iyy="0.00000218412" ixz="0.000000004787" iyz="0.000000000003" izz="0.000004078299" />
+        <mass value="3.16354494"/>
+        <inertia
+              ixx="0.02296002"
+              ixy="0.00000000" iyy="0.04452360"
+              ixz="0.00000000" iyz="-0.00000001" izz="0.02296002"/>
+        <!-- <mass value="${wheel_mass}" />
+        <inertia ixx="0.000002208187" ixy="0.000000000001" iyy="0.00000218412" ixz="0.000000004787" iyz="0.000000000003" izz="0.000004078299" /> -->
       </inertial>
   </link>
